File: RELAY16.sch (EAGLE design)
At the start: 117 parts, among them J1 Analog, J2 POWER, J3 Digital_0_7, J4 M100.1, J5 ICSPPTH, J6 Digital_0_7, J7 PWR SELECT, J8 Digital_0_7, J9 Digital_0_7, Q1 2N7002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

Commit message: Rough draft
Parts:
- removed J1: Analog, freetronics:M06SIP
- removed J2: POWER, freetronics:M08
- removed J3, J8, J9: Digital_0_7, freetronics:M08
- removed J4: M100.1, freetronics-original:M100.1
- removed J5: ICSPPTH, freetronics-jon:ICSPPTH
- removed J7: PWR SELECT, SparkFun:M02PTH
- removed SJ4: (no value), freetronics-jon:SJN
- added IC1: MCP23017SO, microchip:MCP23017SO
- added R51, R52, R53: 10K, freetronics-master-v1:RESISTOR0603
- added R54, R55: 4K7, freetronics-master-v1:RESISTOR0603
- added SJ3: (no value), freetronics-master-v1.1:SJ2W
- J6: value Digital_0_7 -> (none); device freetronics:M08 -> freetronics-master-v1.1:PINHD-2X3
Connections:
- removed net 3V3: J2.4
- removed net 5V: J2.5, SJ4.2
- removed net A0: J1.1
- removed net A1: J1.2
- removed net A2: J1.3
- removed net A3: J1.4
- removed net A4_SDA: J1.5
- removed net A5_SCL: J1.6
- removed net AREF: J4.8
- removed net D0_RX: J3.1
- removed net D10: J4.3
- removed net D11_MOSI: J4.4
- removed net D12_MISO: J4.5
- removed net D13_SCK: J4.6
- removed net D1_TX: J3.2
- removed net D2: J3.3
- removed net D22: J8.8
- removed net D23: J9.8
- removed net D24: J8.7
- removed net D25: J9.7
- removed net D26: J8.6
- removed net D27: J9.6
- removed net D28: J8.5
- removed net D29: J9.5
- removed net D3: J3.4
- removed net D30: J8.4
- removed net D31: J9.4
- removed net D32: J8.3
- removed net D33: J9.3
- removed net D34: J8.2
- removed net D35: J9.2
- removed net D36: J8.1
- removed net D37: J9.1
- removed net D4: J3.5
- removed net D5: J3.6
- removed net D6: J3.7
- removed net D7: J3.8
- removed net D8: J4.1
- removed net D9: J4.2
- removed net N$71: J6.8
- removed net N$72: J6.7
- removed net N$73: J6.6
- removed net N$74: J6.5
- removed net N$75: J6.4
- removed net N$76: J6.3
- removed net N$77: J6.2
- removed net N$78: J6.1
- removed net NC: J2.1
- removed net R3_SCL: J4.10
- removed net R3_SDA: J4.9
- removed net VIN: J2.8, J7.2
- new net ADDR0: IC1.A0, J6.2, R51.2
- new net ADDR1: IC1.A1, J6.4, R52.2
- new net ADDR2: IC1.A2, J6.6, R53.2
- new net GPB0: IC1.GPB0, R28.2
- new net GPB1: IC1.GPB1, R30.2
- new net GPB2: IC1.GPB2, R32.2
- new net GPB3: IC1.GPB3, R34.2
- new net GPB4: IC1.GPB4, R36.2
- new net GPB5: IC1.GPB5, R38.2
- new net GPB6: IC1.GPB6, R40.2
- new net GPB7: IC1.GPB7, R42.2
- new net N$2: R55.2, SJ3.3
- new net N$6: R54.2, SJ3.1
- new net SCL: IC1.SCL, R55.1
- new net SDA: IC1.SDA, R54.1
- net 12V: no longer J7.1
- net GND: now also IC1.VSS, R51.1, R52.1, R53.1; no longer J2.6, J2.7, J4.7
- net GPA0: now also IC1.GPA0; no longer R28.2
- net GPA1: now also IC1.GPA1; no longer R30.2
- net GPA2: now also IC1.GPA2; no longer R32.2
- net GPA3: now also IC1.GPA3; no longer R34.2
- net GPA4: now also IC1.GPA4; no longer R36.2
- net GPA5: now also IC1.GPA5; no longer R38.2
- net GPA6: now also IC1.GPA6; no longer R40.2
- net GPA7: now also IC1.GPA7; no longer R42.2
- net IOREF: now also IC1.VDD, J6.1, J6.3, J6.5, SJ3.2; no longer J2.2, SJ4.1
- net RESET: now also IC1.!RESET; no longer J2.3
Other:
- note added: "(C)2019 SuperHouse Automation Pty Ltd"
- note added: "16-Channel Relay Driver Module"
- note added: "I2C Latch"
- note added: "SKU: RELAY16"
- note added: "ToDo: * Add Seeed header * Power from screw terminals, add 0.1" headers too * Reset? How to handle?"
- note added: "V1.0 (2019-04-04)"
- note added: "www.superhouse.tv/relay16"
- note removed: "(C)2015 Freetronics Pty Ltd: www.freetronics.com"
- note removed: "5V/IOREF Link"
- note removed: "Arduino Headers"
- note removed: "Connect across one side of SJ1 & 2 after other routing"
- note removed: "Freetronics 16-Channel Relay Driver Shield"
- note removed: "ICSP Passthrough"
- note removed: "ICSP passthrough Pull-up cut track Default to R3 headers Use IOREF as VCC"
- note removed: "SKU: RELAY8"
- note removed: "V1.0 (2015-03-09)"
- note removed: "www.freetronics.com/relay8"
- moved on the sheet: D9, JP3
